File: am-radio-backups/rev1.0-180x62/am-radio.kicad_sch (KiCad schematic)
At the start: 51 parts, among them J1 SPEAKER 8R, Q1 2N3904, Q2 2N3904, Q3 2N3904, Q4 2N3904, Q5 2N3904, Q6 2N3904, SW1 POWER, T1 42IF101 (yellow), T2 42IF102 (white), T3 42IF103 (black), T4 42TU013, T5 42TU200

Commit message: checkpoint
Parts:
- BT1: value 3xAAA 4.5V -> 3xAA 4.5V; footprint Battery:BatteryHolder_Keystone_2479_3xAAA -> Battery:BatteryHolder_TruPower_BH-331P_3xAA
- H1, H2, H3, H4: value M2.5 -> M3; footprint MountingHole:MountingHole_2.7mm_M2.5 -> MountingHole:MountingHole_3.2mm_M3
Other:
- note added: "AM BROADCAST RECEIVER - 6 transistor superheterodyne, 455 kHz IF, 4.5 V (3xAA), negative ground, all 2N3904 NPN"
- note removed: "AM BROADCAST RECEIVER - 6 transistor superheterodyne, 455 kHz IF, 4.5 V (3xAAA), negative ground, all 2N3904 NPN"
Changed lines of the file:
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@@
 	(label "DET" (at 129.54 121.92 0) (effects (font (size 1.27 1.27)) (justify left bottom)))
 	(label "DET" (at 227.33 88.9 0) (effects (font (size 1.27 1.27)) (justify left bottom)))
-	(text "AM BROADCAST RECEIVER - 6 transistor superheterodyne, 455 kHz IF, 4.5 V (3xAAA), negative ground, all 2N3904 NPN" (exclude_from_sim no) (at 20.32 40.64 0) (effects (font (size 2.5 2.5)) (justify left bottom)))
+	(text "AM BROADCAST RECEIVER - 6 transistor superheterodyne, 455 kHz IF, 4.5 V (3xAA), negative ground, all 2N3904 NPN" (exclude_from_sim no) (at 20.32 40.64 0) (effects (font (size 2.5 2.5)) (justify left bottom)))
 	(text "Stages:  Q1 converter (mixer + local oscillator, L2 red)  ->  T1 (yellow)  ->  Q2 IF amp with AGC  ->  T2 (white)  ->  Q3 IF amp  ->  T3 (black)  ->  D1 detector  ->  RV1 volume  ->  Q4 driver  ->  T4  ->  Q5/Q6 class-B push-pull  ->  T5  ->  8 ohm speaker" (exclude_from_sim no) (at 20.32 46.99 0) (effects (font (size 1.5 1.5)) (justify left bottom)))
 	(text "Alignment: set VC1 fully closed, adjust L2 slug so the local oscillator is ~985 kHz (station at 530 kHz); at the high end use the VC1 oscillator trimmer for ~2055 kHz (1600 kHz). Peak T1, T2, T3 slugs for max audio on a weak station (they are pre-tuned to 455 kHz). Peak L1 by sliding the coil on the rod at the low end and the VC1 antenna trimmer at the high end. If the oscillator does not start, swap the L2 pin 4/6 feedback leads." (exclude_from_sim no) (at 20.32 156.21 0) (effects (font (size 1.5 1.5)) (justify left bottom)))
@@
 		(dnp no)
 		(property "Reference" "BT1" (at 334.01 135.89 0) (effects (font (size 1.27 1.27)) (justify left)))
-		(property "Value" "3xAAA 4.5V" (at 334.01 138.43 0) (effects (font (size 1.27 1.27)) (justify left)))
-		(property "Footprint" "Battery:BatteryHolder_Keystone_2479_3xAAA" (at 330.2 137.16 0) (effects (font (size 1.27 1.27)) (hide yes)))
+		(property "Value" "3xAA 4.5V" (at 334.01 138.43 0) (effects (font (size 1.27 1.27)) (justify left)))
+		(property "Footprint" "Battery:BatteryHolder_TruPower_BH-331P_3xAA" (at 330.2 137.16 0) (effects (font (size 1.27 1.27)) (hide yes)))
 		(property "Datasheet" "" (at 330.2 137.16 0) (effects (font (size 1.27 1.27)) (hide yes)))
 		(property "Description" "" (at 330.2 137.16 0) (effects (font (size 1.27 1.27)) (hide yes)))
@@
 		(dnp no)
 		(property "Reference" "H1" (at 380 133.35 0) (effects (font (size 1.27 1.27))))
-		(property "Value" "M2.5" (at 380 140.97 0) (effects (font (size 1.27 1.27))))
-		(property "Footprint" "MountingHole:MountingHole_2.7mm_M2.5" (at 380 137.16 0) (effects (font (size 1.27 1.27)) (hide yes)))
+		(property "Value" "M3" (at 380 140.97 0) (effects (font (size 1.27 1.27))))
+		(property "Footprint" "MountingHole:MountingHole_3.2mm_M3" (at 380 137.16 0) (effects (font (size 1.27 1.27)) (hide yes)))
 		(property "Datasheet" "" (at 380 137.16 0) (effects (font (size 1.27 1.27)) (hide yes)))
 		(property "Description" "" (at 380 137.16 0) (effects (font (size 1.27 1.27)) (hide yes)))
@@
 		(dnp no)
 		(property "Reference" "H2" (at 388 133.35 0) (effects (font (size 1.27 1.27))))
-		(property "Value" "M2.5" (at 388 140.97 0) (effects (font (size 1.27 1.27))))
-		(property "Footprint" "MountingHole:MountingHole_2.7mm_M2.5" (at 388 137.16 0) (effects (font (size 1.27 1.27)) (hide yes)))
+		(property "Value" "M3" (at 388 140.97 0) (effects (font (size 1.27 1.27))))
+		(property "Footprint" "MountingHole:MountingHole_3.2mm_M3" (at 388 137.16 0) (effects (font (size 1.27 1.27)) (hide yes)))
 		(property "Datasheet" "" (at 388 137.16 0) (effects (font (size 1.27 1.27)) (hide yes)))
 		(property "Description" "" (at 388 137.16 0) (effects (font (size 1.27 1.27)) (hide yes)))
@@
 		(dnp no)
 		(property "Reference" "H3" (at 396 133.35 0) (effects (font (size 1.27 1.27))))
-		(property "Value" "M2.5" (at 396 140.97 0) (effects (font (size 1.27 1.27))))
-		(property "Footprint" "MountingHole:MountingHole_2.7mm_M2.5" (at 396 137.16 0) (effects (font (size 1.27 1.27)) (hide yes)))
+		(property "Value" "M3" (at 396 140.97 0) (effects (font (size 1.27 1.27))))
+		(property "Footprint" "MountingHole:MountingHole_3.2mm_M3" (at 396 137.16 0) (effects (font (size 1.27 1.27)) (hide yes)))
 		(property "Datasheet" "" (at 396 137.16 0) (effects (font (size 1.27 1.27)) (hide yes)))
 		(property "Description" "" (at 396 137.16 0) (effects (font (size 1.27 1.27)) (hide yes)))
@@
 		(dnp no)
 		(property "Reference" "H4" (at 404 133.35 0) (effects (font (size 1.27 1.27))))
-		(property "Value" "M2.5" (at 404 140.97 0) (effects (font (size 1.27 1.27))))
-		(property "Footprint" "MountingHole:MountingHole_2.7mm_M2.5" (at 404 137.16 0) (effects (font (size 1.27 1.27)) (hide yes)))
+		(property "Value" "M3" (at 404 140.97 0) (effects (font (size 1.27 1.27))))
+		(property "Footprint" "MountingHole:MountingHole_3.2mm_M3" (at 404 137.16 0) (effects (font (size 1.27 1.27)) (hide yes)))
 		(property "Datasheet" "" (at 404 137.16 0) (effects (font (size 1.27 1.27)) (hide yes)))
 		(property "Description" "" (at 404 137.16 0) (effects (font (size 1.27 1.27)) (hide yes)))
